File: KiCad/Spark-AE-PCB/Shock-AE-PCB.kicad_sch (KiCad schematic)
At the start: 16 parts, among them J1 SSM-120-L-SV-BE, J2 SSM-120-L-SV-BE, J3 Conn_02x10_Odd_Even, J4 Conn_02x05_Odd_Even, J5 Conn_01x08_Socket, J6 Conn_01x08_Socket, J7 UJ32-C-V-G-TH-5-P24-TR, SW1 SW_Push, SW2 SW_Push, U1 PJS008U-3000-0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

Commit message: rearranged Shock controls to be aligned and offset with bus connector
Parts:
- removed J1, J2: SSM-120-L-SV-BE, clectric-diy:SAMTEC_SSM-120-L-SV-BE, symbol clectric-diy:SSM-120-L-SV-BE
- removed J3: Conn_02x10_Odd_Even, Connector_PinHeader_2.54mm:PinHeader_2x10_P2.54mm_Vertical, symbol Connector_Generic:Conn_02x10_Odd_Even
- removed J7: UJ32-C-V-G-TH-5-P24-TR, clectric-diy:SAMESKY_UJ32-C-V-G-TH-5-P24-TR, symbol clectric-diy:UJ32-C-V-G-TH-5-P24-TR
- removed U1: PJS008U-3000-0, clectric-diy:PJS008U-3000-0, symbol clectric-diy:PJS008U-3000-0
- added J1, J2: Conn_01x20_Pin, symbol Connector:Conn_01x20_Pin
Connections:
- net +3V3_A: now also J2.1 (Pin_1)
- net +3V3_D: now also J2.18 (Pin_18)
- net A1_D16: now also J2.3 (Pin_3)
- net A7_D22: now also J2.9 (Pin_9)
- net AUDIO_IN_1: now also J1.16 (Pin_16)
- net AUDIO_IN_2: now also J1.17 (Pin_17)
- net AUDIO_OUT_1: now also J1.18 (Pin_18)
- net AUDIO_OUT_2: now also J1.19 (Pin_19)
- net ENC_A: now also J2.13 (Pin_13)
- net ENC_B: now also J2.12 (Pin_12)
- net ENC_CLICK: now also J1.14 (Pin_14)
- net GND: now also J1.20 (Pin_20), J2.20 (Pin_20)
- net I2C_SCL: now also J1.12 (Pin_12)
- net I2C_SDA: now also J1.13 (Pin_13)
- net LED_1_B: now also J2.5 (Pin_5)
- net LED_1_G: now also J2.6 (Pin_6)
- net LED_1_R: now also J2.7 (Pin_7)
- net LED_2_B: now also J2.10 (Pin_10)
- net LED_2_G: now also J2.11 (Pin_11)
- net LED_2_R: now also J2.4 (Pin_4)
- net POT_1: now also J2.8 (Pin_8)
- net POT_2: now also J2.2 (Pin_2)
- net SD_CK: now also J1.7 (Pin_7)
- net SD_CMD: now also J1.6 (Pin_6)
- net SD_D0: now also J1.5 (Pin_5)
- net SD_D1: now also J1.4 (Pin_4)
- net SD_D2: now also J1.3 (Pin_3)
- net SD_D3: now also J1.2 (Pin_2)
- net SPI_MISO: now also J1.10 (Pin_10)
- net SPI_MOSI: now also J1.11 (Pin_11)
- net SPI_NSS: now also J1.8 (Pin_8)
- net SPI_SCK: now also J1.9 (Pin_9)
- net TAC_SWITCH_1: now also J2.14 (Pin_14)
- net TAC_SWITCH_2: now also J2.15 (Pin_15)
- net USART1_RX: now also J1.15 (Pin_15)
- net USB_OTG_FS_D+: now also J2.17 (Pin_17)
- net USB_OTG_FS_D-: now also J2.16 (Pin_16)
- net USB_OTG_FS_ID: now also J1.1 (Pin_1)
- net VIN: now also J2.19 (Pin_19)
Other:
- title: Spark-AE-Upper -> Shock-AE-PCB
