File: KiCad/Shock-AE-PCB/Shock-AE-PCB.kicad_sch (KiCad schematic)
At the start: 39 parts, among them J1 Conn_01x08_Socket, J2 Conn_01x08_Socket, J3 Conn_01x20_Pin, J4 Conn_01x20_Pin, J5 Conn_02x05_Odd_Even, SW1 SW_Push, SW2 SW_Push, U1 WS2811, U2 Daisy_Seed

Commit message: retracing to seperate analog and digital gnd
Parts:
- added J6: Conn_02x05_Odd_Even, Connector_PinHeader_2.54mm:PinHeader_2x05_P2.54mm_Vertical, symbol Connector_Generic:Conn_02x05_Odd_Even
Connections:
- net +3V3_A: now also J6.1 (Pin_1)
- net +3V3_D: now also J6.2 (Pin_2)
- net +5V: now also U1.8 (VDD)
- net A1_D16: now also D15.2 (A), D7.1 (K); no longer D15.1 (K), D7.2 (A)
- net A7_D22: now also D16.2 (A), D8.1 (K); no longer D16.1 (K), D8.2 (A)
- net AUDIO_IN_1: now also D1.1 (K); no longer D1.2 (A)
- net AUDIO_IN_2: now also D2.1 (K); no longer D2.2 (A)
- net AUDIO_OUT_1: now also D9.2 (A); no longer D9.1 (K)
- net AUDIO_OUT_2: now also D10.2 (A); no longer D10.1 (K)
- net GND: now also J6.3 (Pin_3), J6.4 (Pin_4)
- net I2C_SCL: now also J6.6 (Pin_6)
- net I2C_SDA: now also J6.5 (Pin_5)
- net LED_1_B: now also LED1.4, R3.2
- net LED_1_G: now also LED1.1, R1.2
- net LED_1_R: now also LED1.2, R2.2
- net LED_2_B: now also LED2.4, R6.2
- net LED_2_G: now also LED2.1, R4.2
- net LED_2_R: now also LED2.2, R5.2
- net POT_1_CV: now also D5.1 (K); no longer D3.2 (A)
- net POT_2_CV: now also D6.1 (K); no longer D4.2 (A)
- net SPI_MISO: now also J6.8 (Pin_8)
- net SPI_MOSI: now also U1.6 (DIN), J6.7 (Pin_7)
- net SPI_NSS: now also J6.9 (Pin_9)
- net SPI_SCK: now also J6.10 (Pin_10)
- net at J1.3: now also D3.2 (A); no longer D3.1 (K)
- net at J1.1: now also D1.2 (A); no longer D1.1 (K)
- net at J1.2: now also D2.2 (A); no longer D2.1 (K)
- net at J1.4: now also D4.2 (A); no longer D4.1 (K)
- net at J1.5: now also D5.2 (A); no longer D5.1 (K)
- net at J1.6: now also D6.2 (A); no longer D6.1 (K)
- net at J1.7: now also D7.2 (A); no longer D7.1 (K)
- net at J1.8: now also D8.2 (A); no longer D8.1 (K)
- net at D11.1 (K): now also J2.3
- net at D11.2 (A): no longer J2.3
- net at J2.8: now also D16.1 (K); no longer D16.2 (A)
- net at J2.1: now also D9.1 (K); no longer D9.2 (A)
- net at J2.2: now also D10.1 (K); no longer D10.2 (A)
- net at J2.4: now also D12.1 (K); no longer D12.2 (A)
- net at J2.5: now also D13.1 (K); no longer D13.2 (A)
- net at J2.6: now also D14.1 (K); no longer D14.2 (A)
- net at J2.7: now also D15.1 (K); no longer D15.2 (A)
- net USART1_RX renamed MIDI
- new net SW2_2_CV: D4.1 (K)
- new net SW_1_CV: D3.1 (K)
- no-connect marks 6 -> 8
Other:
- moved on the sheet: D1, D10, D11, D12, D13, D14, D15, D16, D2, D4, D5, D6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

Commit message: partiallly retraced. time for bed.
Parts:
- ENC1: value PEL12T-4225S-S1024 -> ENC
Connections:
- net ENC_RED: now reaches R7.2, U1.1 (OUTR)
- net ENC_GREEN: now reaches R8.2, U1.2 (OUTG)
- net ENC_GREEN: now also ENC1.2 (-_2), R8.1
- net ENC_BLUE: now reaches R9.2, U1.3 (OUTB)
- net ENC_BLUE: now also ENC1.4 (+_1), R9.1
Changed lines of the file:
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@@
 		)
 	)
+	(label "ENC_BLUE"
+		(at 60.96 176.53 0)
+		(effects
+			(font
+				(size 1.27 1.27)
+			)
+			(justify left bottom)
+		)
+	)
+	(label "ENC_GREEN"
+		(at 66.04 171.45 180)
+		(effects
+			(font
+				(size 1.27 1.27)
+			)
+			(justify right bottom)
+		)
+	)
 	(label "LED_1_B"
 		(at 57.15 102.87 180)
@@
 		)
 	)
+	(label "ENC_RED"
+		(at 82.55 168.91 180)
+		(effects
+			(font
+				(size 1.27 1.27)
+			)
+			(justify right bottom)
+		)
+	)
 	(label "LED_2_G"
 		(at 96.52 91.44 0)
@@
 		)
 	)
+	(label "ENC_GREEN"
+		(at 66.04 171.45 180)
+		(effects
+			(font
+				(size 1.27 1.27)
+			)
+			(justify right bottom)
+		)
+	)
+	(label "ENC_GREEN"
+		(at 82.55 171.45 180)
+		(effects
+			(font
+				(size 1.27 1.27)
+			)
+			(justify right bottom)
+		)
+	)
+	(label "ENC_BLUE"
+		(at 82.55 173.99 180)
+		(effects
+			(font
+				(size 1.27 1.27)
+			)
+			(justify right bottom)
+		)
+	)
 	(label "LED_2_R"
 		(at 96.52 97.79 0)
@@
 		)
 	)
+	(label "ENC_BLUE"
+		(at 82.55 173.99 180)
+		(effects
+			(font
+				(size 1.27 1.27)
+			)
+			(justify right bottom)
+		)
+	)
+	(label "ENC_RED"
+		(at 82.55 168.91 180)
+		(effects
+			(font
+				(size 1.27 1.27)
+			)
+			(justify right bottom)
+		)
+	)
+	(label "ENC_BLUE"
+		(at 60.96 176.53 0)
+		(effects
+			(font
+				(size 1.27 1.27)
+			)
+			(justify left bottom)
+		)
+	)
+	(label "ENC_GREEN"
+		(at 82.55 171.45 180)
+		(effects
+			(font
+				(size 1.27 1.27)
+			)
+			(justify right bottom)
+		)
+	)
 	(label "LED_1_G"
 		(at 57.15 92.71 180)
@@
 			)
 		)
-		(property "Value" "PEL12T-4225S-S1024"
+		(property "Value" "ENC"
 			(at 35.56 193.04 90)
 			(effects

Commit message: as expected, AE-1U is too small to squeeze a full Daisy Pod clone (see desc)
This will be the final commit of an attempt to squeeze the full clone onto the AE-1U "Shock". I am moving now to make it an AE-2U called the "Spark".

I plan to come back around to make the "Shock" a slimmed down version of the "Spark" in an AE-1U size.
Parts:
- removed J1, J2: Conn_01x08_Socket, clectric-diy:801-87-008-10-005101, symbol clectric-diy:801-87-008-10-005101
- removed R7, R8, R9: R, Resistor_SMD:R_0402_1005Metric, symbol clectric-diy:CR0603-FX-1001ELF
- removed U2: Daisy_Seed, clectric-diy:DAISY_SEED, symbol clectric-diy:Daisy_Seed
- added C1, C2, C3: 10nF, Capacitor_SMD:C_0402_1005Metric, symbol Device:C
- added D17, D18: D, Diode_SMD:D_0402_1005Metric, symbol Device:D
- added J1, J2: Conn_01x09_Socket, Connector_PinSocket_2.54mm:PinSocket_1x09_P2.54mm_Vertical, symbol Connector:Conn_01x09_Socket
- added NT1: NetTie, NetTie:NetTie-3_SMD_Pad0.5mm, symbol Device:NetTie_3
- added R10, R11, R12, R7, R8, R9: 10K, Resistor_SMD:R_0402_1005Metric, symbol Device:R
- added U3: Daisy_Seed, clectric-diy:DAISY_SEED, symbol clectric-diy:Daisy_Seed
- ENC1: value ENC -> PEL12T-4225S-S1024
- LED1, LED2: value LED-SMD_4P-L1.6-W1.5-BL_A-SP1943B1GHR6C-C01-2T -> A-SP1943B1GHR6C-C01-2T
- R1, R2, R4, R5: value R -> 150R
- R3, R6: value R -> 330R
Connections:
- net +3V3_A: now also U3.21 (3V3_A)
- net +3V3_D: now also R10.2, R11.2, R9.2, U3.38 (3V3_D)
- net +5V: now also U3.39 (VIN)
- net A1_D16: now also D8.1 (K), D17.2 (A), U3.23 (D16); no longer D15.2 (A), D7.1 (K)
- net A7_D22: now also D9.1 (K), D18.2 (A), U3.29 (D22); no longer D16.2 (A), D8.1 (K)
- net AUDIO_IN_1: now also U3.16 (AUDIO_IN_1)
- net AUDIO_IN_2: now also U3.17 (AUDIO_IN_2)
- net AUDIO_OUT_1: now also D10.2 (A), U3.18 (AUDIO_OUT_1); no longer D9.2 (A)
- net AUDIO_OUT_2: now also D11.2 (A), U3.19 (AUDIO_OUT_2); no longer D10.2 (A)
- net ENC_A: now also R7.2, U3.33 (D26); no longer ENC1.A1
- net ENC_B: now also R8.2, U3.32 (D25); no longer ENC1.B1
- net ENC_CLICK: now also R12.2, U3.14 (D13); no longer ENC1.3 (COM)
- net ENC_RED: now also ENC1.1 (-_1)
- net GND: now also NT1.3; no longer ENC1.C1, ENC1.MH1, ENC1.MH2, J3.20 (Pin_20), J4.20 (Pin_20), J6.3 (Pin_3), J6.4 (Pin_4), POT1.1, POT1.4 (EH), POT1.5 (EH), POT2.1, POT2.4 (EH), POT2.5 (EH), SW1.2, SW2.2, U1.4 (GND)
- net I2C_SCL: now also J6.5 (Pin_5), U3.12 (D11); no longer J6.6 (Pin_6)
- net I2C_SDA: now also J6.6 (Pin_6), U3.13 (D12); no longer J6.5 (Pin_5)
- net LED_1_B: now also LED1.2, R2.1, R2.2, U3.25 (D18); no longer LED1.4, R3.1, R3.2
- net LED_1_G: now also U3.26 (D19)
- net LED_1_R: now also LED1.4, R3.1, R3.2, U3.27 (D20); no longer LED1.2, R2.1, R2.2
- net LED_2_B: now also LED2.2, R5.1, R5.2, U3.30 (D23); no longer LED2.4, R6.1, R6.2
- net LED_2_G: now also U3.31 (D24)
- net LED_2_R: now also LED2.4, R6.1, R6.2, U3.24 (D17); no longer LED2.2, R5.1, R5.2
- net POT_1: now also U3.28 (D21)
- net POT_2: now also U3.22 (D15)
- net SD_CK: now also U3.7 (D6)
- net SD_CMD: now also U3.6 (D5)
- net SD_D0: now also U3.5 (D4)
- net SD_D1: now also U3.4 (D3)
- net SD_D2: now also U3.3 (D2)
- net SD_D3: now also U3.2 (D1)
- net SPI_MISO: now also J6.10 (Pin_10), U3.10 (D9); no longer J6.8 (Pin_8)
- net SPI_MOSI: now also J6.8 (Pin_8), U3.11 (D10); no longer J6.7 (Pin_7)
- net SPI_NSS: now also J6.7 (Pin_7), U3.8 (D7); no longer J6.9 (Pin_9)
- net SPI_SCK: now also J6.9 (Pin_9), U3.9 (D8); no longer J6.10 (Pin_10)
- net TAC_SWITCH_1: now also U3.34 (D27)
- net TAC_SWITCH_2: now also U3.35 (D28)
- net USB_OTG_FS_D+: now also U3.37 (D30)
- net USB_OTG_FS_D-: now also U3.36 (D29)
- net USB_OTG_FS_ID: now also U3.1 (D0)
- net MIDI renamed D14
- net D14: now also D16.2 (A), D7.1 (K), U3.15 (D14)
- net POT_1_CV renamed POT1_CV
- net POT_2_CV renamed POT2_CV
- net SW2_2_CV renamed SW2_CV
- net SW_1_CV renamed SW1_CV
- new net: C1.1, ENC1.A1, R7.1, R9.1
- new net: C3.1, ENC1.3 (COM), R11.1, R12.1
- new net: C2.1, ENC1.B1, R10.1, R8.1
- new net AGND: J4.20 (Pin_20), J6.3 (Pin_3), NT1.2, POT1.1, POT1.4 (EH), POT1.5 (EH), POT2.1, POT2.4 (EH), POT2.5 (EH), SW1.2, SW2.2, U3.20 (AGND)
- new net DGND: C1.2, C2.2, C3.2, ENC1.C1, ENC1.MH1, ENC1.MH2, J3.20 (Pin_20), J6.4 (Pin_4), NT1.1, U1.4 (GND), U3.40 (DGND)
- no-connect marks 8 -> 6
Other:
- moved on the sheet: D1, D10, D11, D12, D13, D14, D15, D16, D2, D3, D4, D5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
